File: picofusion.kicad_pcb (KiCad board)
At the start: 4 copper layers, 16 x 16 mm, 45 parts, among them J1 EAST, J2 WEST, J3 SOUTH, J4 NORTH, U1 W25Q16, U2 RP2040, U3 TLV71333PDQNT, U4 ICM42605, U5 BMM150, U6 ICP20100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

Commit message: a little more work
Parts:
- removed C21: 0.1uF, Capacitor_SMD:C_0402_1005Metric
- removed D1: WS2812B-2020, LED_SMD_Extra:WS2812B-2020
- added R8: 2.7K, Resistor_SMD:R_0402_1005Metric, F.Cu at (147.6, 35.6)
- added R9: 2.7K, Resistor_SMD:R_0402_1005Metric, F.Cu at (148.6, 35.6)
- C12: value 0.1uF -> 1uF
- C20: value 0.1uF -> 10uF
- U5: value BMM150 -> MMC5983MA; footprint Package_CSP:WLCSP-12_1.56x1.56mm_P0.4mm -> Package_LGA:LGA-16_3x3mm_P0.5mm
- moved R1 105.9 mm to (161.3, 48.7)
- moved C11 103.2 mm to (161.8, 47.1), turned to 90 degrees
- moved R5 47.2 mm to (154.0, 48.7), turned to 180 degrees
- moved R4 46.7 mm to (152.0, 48.7)
- moved C2 37.5 mm to (158.4, 48.7), turned to 0 degrees
- moved C9 36.6 mm to (156.4, 48.7), turned to 180 degrees
- moved R6 36.3 mm to (152.2, 35.0)
- moved D2 36.3 mm to (150.1, 35.0), turned to 180 degrees
- moved C20 24.2 mm to (151.4, 38.7), turned to 90 degrees
- moved U6 22.8 mm to (160.3, 35.8)
- moved U5 21.8 mm to (148.8, 38.5)
- moved C23 20.0 mm to (158.0, 36.8), turned to 180 degrees
- moved C22 19.9 mm to (158.4, 35.3), turned to 90 degrees
- moved U3 14.5 mm to (157.1, 35.3), turned to 90 degrees
- moved C14 14.4 mm to (155.8, 35.8)
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Connections:
- C12 pad 1: +3V3 -> GND
- C12 pad 2: GND -> +3V3
- C20 pad 1: GND -> Net-(C20-Pad1)
- C20 pad 2: +3V3 -> GND
- U2 pad 5: /SPI0_POCI -> /SPI0_PICO
- U4 pad 1: /SPI0_MISO -> /SPI0_POCI
- U4 pad 14: /SPI0_MOSI -> /SPI0_PICO
Routing:
- net /I2C0_SCL: track 0.73 -> 16.1 mm, vias 0 -> 2
- net /I2C0_SDA: track 0.00 -> 14.8 mm, vias 0 -> 2
- net /SPI0_nCS: track 0.00 -> 13.6 mm, vias 0 -> 3
- net +3V3: track 10.6 -> 22.8 mm, vias 1 -> 0
- net /SPI0_PICO: track 0.00 -> 9.53 mm, vias 0 -> 2
- net /SPI0_SCK: track 0.00 -> 8.72 mm, vias 0 -> 2
- net /XOUT: track 2.18 -> 10.6 mm, vias 0 -> 2
- net /XIN: track 1.58 -> 9.49 mm
- net /SPI0_POCI: track 0.00 -> 7.75 mm, vias 0 -> 1
- net GND: track 3.63 -> 8.87 mm, vias 0 -> 4
- net Net-(D2-Pad1): track 0.00 -> 3.19 mm
- net +1V1: track 3.58 -> 6.17 mm
- net /DRDY_ICM42605: track 0.00 -> 2.47 mm, vias 0 -> 2
- net /USB_MCU_DN: track 0.00 -> 1.73 mm
- net /USB_MCU_DP: track 0.00 -> 1.73 mm
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Other:
- board size 16 x 16 mm -> 18 x 18 mm
