File: peripherals.kicad_sch (KiCad schematic)
At the start: 13 parts, among them U7 TJA1051TK-3, U8 74LVC1T45GS

Commit message: schematic: more improvements towards R3
Parts:
- C27, C28, C29: value 0.1uF -> 0u1
- C30: value 0.1uF -> 0u1; footprint Capacitor_SMD:C_0201_0603Metric -> Capacitor_SMD:C_0402_1005Metric
- C31: value 1uF -> 1u; footprint Capacitor_SMD:C_0201_0603Metric -> Capacitor_SMD:C_0402_1005Metric
Other:
- company: (none) -> Kalyan S, Vincent W, Kai G
- moved on the sheet: R11

Commit message: schematic: refresh sensors, mcu and redo pinout
    * update rp2040 -> rp2350b
    * update icm-42688p -> icm-45686
    * update bmm150 -> bmm350
    * add current sensing logic
    * change pinout count and update pinout
    * drop led and heater support
    * add can termination
Parts:
- removed C29: 0u1, Capacitor_SMD:C_0201_0603Metric, symbol Device:C
- removed C30: 0u1, Capacitor_SMD:C_0402_1005Metric, symbol Device:C
- removed C31: 1u, Capacitor_SMD:C_0402_1005Metric, symbol Device:C_Small
- removed D4: WS2812B-2020, LED_SMD_Extra:WS2812B-2020, symbol LED_Extra:WS2812B-2020
- removed U8: 74LVC1T45GS, 74LVC1T45:PSON35P100X100X35-6N, symbol 74LVC1T45:74LVC1T45GS
- added D4, D6: BLUE, symbol Device:LED
- added D5: RED, symbol Device:LED
- added Q1: NMOS, symbol Simulation_SPICE:NMOS
- added R23, R7: 1K5, symbol Device:R
- added R25: 120, symbol Device:R
- added R26: 10K, symbol Device:R
- C27, C28: value 0u1 -> 100n
- R10, R12, R13: now not fitted
- R14: value 10K -> 1K5; footprint Resistor_SMD:R_0402_1005Metric -> (none)
- U7: value TJA1051TK-3 -> TJA1051TK/3/1J
Connections:
- net +3V3: no longer R14.1
- net CAN_N: now also Q1.3 (S)
- net CAN_P: now also R25.1
- net GND: now also R14.2, R23.2, R26.2, R7.2
- new net: D6.1 (K), R23.1
- new net: D4.1 (K), R7.1
- new net: D5.1 (K), R14.1
- new net: Q1.1 (D), R25.2
- new net CAN_TERM: Q1.2 (G), R26.1
- new net LED_ACT: D4.2 (A)
- new net LED_B/E: D5.2 (A)
- new net LED_PWR: D6.2 (A)
Other:
- note added: "CAN Termination Resistor"
- note added: "Status LEDs"
- note added: "TODO: identify parts and check resistances"
- note removed: "3V3->5V Level Shifter"
- note removed: "Neopixel Serial LED"
- note removed: "Onboard Neopixel"
- moved on the sheet: C27, C28, R11, U7

Commit message: schematic: footprint assignment
Parts:
- D4, D5, D6: footprint (none) -> LED_SMD:LED_0402_1005Metric
- R10, R11: footprint Resistor_SMD:R_0402_1005Metric -> Resistor_SMD:R_0201_0603Metric
- R14, R23, R25, R7: footprint (none) -> Resistor_SMD:R_0402_1005Metric
- R26: footprint (none) -> Resistor_SMD:R_0201_0603Metric
Changed lines of the file:
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@@
 			)
 		)
-		(property "Footprint" ""
+		(property "Footprint" "LED_SMD:LED_0402_1005Metric"
 			(at 41.91 64.77 0)
 			(effects
@@
 			)
 		)
-		(property "Footprint" "Resistor_SMD:R_0402_1005Metric"
+		(property "Footprint" "Resistor_SMD:R_0201_0603Metric"
 			(at 90.932 48.26 90)
 			(effects
@@
 			)
 		)
-		(property "Footprint" ""
+		(property "Footprint" "LED_SMD:LED_0402_1005Metric"
 			(at 41.91 36.83 0)
 			(effects
@@
 			)
 		)
-		(property "Footprint" ""
+		(property "Footprint" "LED_SMD:LED_0402_1005Metric"
 			(at 41.91 50.8 0)
 			(effects
@@
 			)
 		)
-		(property "Footprint" ""
+		(property "Footprint" "Resistor_SMD:R_0402_1005Metric"
 			(at 52.07 38.608 90)
 			(effects
@@
 			)
 		)
-		(property "Footprint" ""
+		(property "Footprint" "Resistor_SMD:R_0402_1005Metric"
 			(at 52.07 66.548 90)
 			(effects
@@
 			)
 		)
-		(property "Footprint" ""
+		(property "Footprint" "Resistor_SMD:R_0402_1005Metric"
 			(at 228.092 41.91 90)
 			(effects
@@
 			)
 		)
-		(property "Footprint" ""
+		(property "Footprint" "Resistor_SMD:R_0402_1005Metric"
 			(at 52.07 52.578 90)
 			(effects
@@
 			)
 		)
-		(property "Footprint" ""
+		(property "Footprint" "Resistor_SMD:R_0201_0603Metric"
 			(at 217.932 59.69 90)
 			(effects
@@
 			)
 		)
-		(property "Footprint" "Resistor_SMD:R_0402_1005Metric"
+		(property "Footprint" "Resistor_SMD:R_0201_0603Metric"
 			(at 90.932 60.96 90)
 			(effects
